Commit message: fixed Fetch and UR collision tags

File: Assets/Robotics/fetch.urdf (robot description, URDF)
Before this commit: robot fetch, 16 links, 15 joints
Links:
- added link bellows_link2, mass 0.169374038216602; collision mesh filename=package://Models/fetch/bellows_link_collision.STL; visual mesh filename=package://Models/fetch/bellows_link.STL
- added link estop_link, mass 0.00196130439134723; collision mesh filename=package://Models/fetch/estop_link.STL; visual mesh filename=package://Models/fetch/estop_link.dae
- added link l_wheel_link, mass 4.3542; collision mesh filename=package://Models/fetch/l_wheel_link_collision.STL; visual mesh filename=package://Models/fetch/l_wheel_link.STL
- added link r_wheel_link, mass 4.3542; collision mesh filename=package://Models/fetch/r_wheel_link_collision.STL; visual mesh filename=package://Models/fetch/r_wheel_link.STL
- link fetch_base_link: mass None -> 70.1294
Joints:
- added joint bellows_joint2: type fixed, parent torso_lift_link, child bellows_link2, origin xyz=0 0 0 rpy=0 0 0
- added joint estop_joint: type fixed, parent fetch_base_link, child estop_link, origin xyz=-0.12465 0.23892 0.31127 rpy=1.5708 0 0, axis 0 0 0
- added joint l_wheel_joint: type continuous, parent fetch_base_link, child l_wheel_link, origin xyz=0.0012914 0.18738 0.055325 rpy=-6.123E-17 0 0, axis 0 1 0, limit effort=8.85 velocity=17.4
- added joint r_wheel_joint: type continuous, parent fetch_base_link, child r_wheel_link, origin xyz=0.0012914 -0.18738 0.055325 rpy=-6.123E-17 0 0, axis 0 1 0, limit effort=8.85 velocity=17.4
