Commit message: fixed Fetch hand-guided actuation

File: Assets/Robotics/fetch_borked.urdf (robot description, URDF)
Before this commit: robot fetch, 16 links, 15 joints
Links:
- added link estop_link, mass 0.00196130439134723; collision mesh filename=package://Models/fetch/estop_link.STL; visual mesh filename=package://Models/fetch/estop_link.dae
Joints:
- added joint estop_joint: type fixed, parent fetch_base_link, child estop_link, origin xyz=-0.12465 0.23892 0.31127 rpy=1.5708 0 0, axis 0 0 0
